File: robot-dev-board-2026.kicad_sch (KiCad schematic)
At the start: 4 parts, among them U1 RP2040, U2 MIC4426

Commit message: initial Branch commit
Parts:
- added U3: MCP14A0304xMNY, Package_DFN_QFN:WDFN-8-1EP_3x2mm_P0.5mm_EP1.3x1.4mm, symbol Driver_FET:MCP14A0304xMNY
Connections:
- new net: U3.3 (GND), U3.9 (GND)
Changed lines of the file:
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@@
+		)
+	)
+	(symbol
+		(lib_id "Driver_FET:MCP14A0304xMNY")
+		(at 54.61 130.81 0)
+		(unit 1)
+		(exclude_from_sim no)
+		(in_bom yes)
+		(on_board yes)
+		(dnp no)
+		(fields_autoplaced yes)
+		(property "Reference" "U3"
+			(at 56.7533 118.11 0)
+			(effects
+				(font
+					(size 1.27 1.27)
+				)
+				(justify left)
+			)
+		)
+		(property "Value" "MCP14A0304xMNY"
+			(at 56.7533 120.65 0)
+			(effects
+				(font
+					(size 1.27 1.27)
+				)
+				(justify left)
+			)
+		)
+		(property "Footprint" "Package_DFN_QFN:WDFN-8-1EP_3x2mm_P0.5mm_EP1.3x1.4mm"
+			(at 54.61 111.76 0)
+			(effects
+				(font
+					(size 1.27 1.27)
+				)
+				(hide yes)
+			)
+		)
+		(property "Datasheet" "http://ww1.microchip.com/downloads/en/DeviceDoc/MCP14A0303_4_5-Data-Sheet-20006046A.pdf"
+			(at 54.61 138.43 0)
+			(effects
+				(font
+					(size 1.27 1.27)
+				)
+				(hide yes)
+			)
+		)
+		(property "Description" "Dual 3A-Peak MOSFET Driver, non-inverting outputs, DFN-8"
+			(at 54.61 130.81 0)
+			(effects
+				(font
+					(size 1.27 1.27)
+				)
+				(hide yes)
+			)
+		)
+		(pin "5"
+		)
+		(pin "2"
+		)
+		(pin "1"
+		)
+		(pin "8"
+		)
+		(pin "4"
+		)
+		(pin "7"
+		)
+		(pin "3"
+		)
+		(pin "9"
+		)
+		(pin "6"
+		)
+		(instances
+			(project ""
+				(path "/bf523f8d-75d7-479b-b431-b3dab10d93ee"
+					(reference "U3")
+					(unit 1)
+				)
+			)
 		)
 	)
