File: robot-dev-board-2026.kicad_sch (KiCad schematic)
At the start: 25 parts, among them J1 USB_C_Receptacle_USB2.0_16P, J10 6V_Out_1, J11 6V_Out_2, J12 6V_Out_3, J13 6V_Out_4, J14 6V_Out_5, J15 6V_Out_6, J2 Out_1, J3 Out_2, J4 Out_3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

Commit message: Updated Schematic
Parts:
- added 10k1, 1k1: R_Small, symbol Device:R_Small
- added D1: 1N4148, Diode_THT:D_DO-35_SOD27_P12.70mm_Horizontal, symbol Diode:1N4148
- added D2: GREEN, LED_SMD:LED_0201_0603Metric, symbol Device:LED
- added J16, J17, J18, J19: ADCX, symbol Connector_Generic:Conn_01x03
- added LS1: 3000Hz, symbol Device:Speaker
- added Q1: Q_NPN, symbol Device:Q_NPN
- added R3: 180Ω, symbol Device:R_Small
- added RX1: TX, symbol Connector_Generic:Conn_01x02
- added SW2: SW_Push, symbol Switch:SW_Push
- added U4: L293D, Package_DIP:DIP-16_W7.62mm, symbol Driver_Motor:L293D
- renumbered 0.1u to 0.1u1, 0.33u to 0.33u1, 10µF to 10µF1
Connections:
- net +3V3 is gone; now on net +3.3V: 10µF1.2, U2.2 (VOUT), U2.4 (VOUT)
- net +3.3V: now also D1.1 (K), J16.2 (Pin_2), J17.2 (Pin_2), J18.2 (Pin_2), J19.2 (Pin_2), LS1.1
- net GND: now also 1k1.2, J16.1 (Pin_1), J17.1 (Pin_1), J18.1 (Pin_1), J19.1 (Pin_1), Q1.E, SW2.1
- new net: 10k1.1, SW2.2
- new net: D1.2 (A), LS1.2, Q1.C
- new net: 1k1.1, D2.1 (K)
- new net: Q1.B, R3.2
- new net GPIO_0: RX1.2 (Pin_2)
- new net GPIO_1: RX1.1 (Pin_1)
- new net GPIO_XX: 10k1.2, D2.2 (A)
- new net GPIO_XX_ADCX: J16.3 (Pin_3), J17.3 (Pin_3), J18.3 (Pin_3), J19.3 (Pin_3)
Other:
- note added: "ADC"
- note added: "LED"
- note added: "RX/TX"
- note added: "Speaker"
- note added: "Stop-Start Switch"
